Commit message: Four bar linkage modelled with trajopt constraints

File: wire_cutting/urdf/irb6400r.xacro (robot description, xacro)
@@ -1,5 +1,5 @@
 <?xml version="1.0" ?>
 <robot name="irb6400r" xmlns:xacro="http://ros.org/wiki/xacro">
-  <xacro:include filename="$(find wire_cutting)/urdf/irb6400r_macro.xacro"/>
+  <xacro:include filename="$(find wire_cutting)/urdf/irb6400r_macro_parallel.xacro"/>
   <xacro:irb6400r prefix=""/>
 </robot>

File: wire_cutting/urdf/irb6400r_macro_parallel.xacro (robot description, xacro)
@@ -63,4 +63,6 @@
       </visual>
     </link>
+    <link name="${prefix}link_p"> <!-- Virtual link related to four bar linkage -->
+    </link>
     <link name="${prefix}link_4">
       <collision name="collision">
@@ -118,36 +120,4 @@
       </collision>
     </link>
-    <!--Cylinder and piston -->
-    <!--link name="${prefix}link_cylinder">
-      <collision name="collision">
-        <geometry>
-          <mesh filename="package://wire_cutting/meshes/irb6400r/collision/cylinder.stl"/>
-        </geometry>
-        <material name="yellow"/>
-      </collision>
-      <visual name="visual">
-        <geometry>
-          <mesh filename="package://wire_cutting/meshes/irb6400r/visual/cylinder.stl"/>
-        </geometry>
-        <material name="orange"/>
-      </visual>
-    </link>
-    <link name="${prefix}link_piston">
-      <collision name="collision">
-        <geometry>
-          <mesh filename="package://wire_cutting/meshes/irb6400r/collision/piston.stl"/>
-        </geometry>
-        <material name="yellow"/>
-      </collision>
-      <visual name="visual">
-        <geometry>
-          <mesh filename="package://wire_cutting/meshes/irb6400r/visual/piston.stl"/>
-        </geometry>
-        <material name="orange"/>
-      </visual>
-    </link> -->
-    <!-- end of link list -->
-    <!-- joint list -->
-    <!-- TODO update limits and velocities (bar linkage between axis 2 and 3!)-->
     <joint type="revolute" name="${prefix}joint_1">
       <origin xyz="0 0 0.27" rpy="0 0 0"/>
@@ -164,8 +134,16 @@
       <limit effort="0" lower="-1.22" upper="1.48" velocity="1.22"/>
     </joint>
-    <joint type="revolute" name="${prefix}joint_3">
+    <joint type="revolute" name="${prefix}joint_p"> <!-- Virtualt joint related to four bar linkage -->
       <origin xyz="0 0 1.05" rpy="0 0 0"/>
       <axis xyz="0 1 0"/>
       <parent link="${prefix}link_2"/>
+      <child link="${prefix}link_p"/>
+      <limit effort="0" lower="-1.48" upper="1.22" velocity="1.22"/>
+      <!--<mimic joint="${prefix}joint_2" multiplier="-1" offset="0" /> Mimic not used, constraints instead-->
+    </joint>
+    <joint type="revolute" name="${prefix}joint_3">
+      <origin xyz="0 0 0" rpy="0 0 0"/>
+      <axis xyz="0 1 0"/>
+      <parent link="${prefix}link_p"/>
       <child link="${prefix}link_3"/>
       <limit effort="0" lower="-0.489" upper="1.92" velocity="1.22"/>
@@ -203,19 +181,4 @@
       <origin xyz="0 0 1.861" rpy="0 0 0"/>
     </joint>
-    <!--<joint type="fixed" name="${prefix}joint_cylinder">
-      <origin xyz="-0.365 -0.1895 0.405" rpy="0 -0.170 0"/>
-      <axis xyz="0 1 0"/>
-      <parent link="${prefix}link_1"/>
-      <child link="${prefix}link_cylinder"/>
-      <limit effort="0" lower="-2.96705973" upper="2.96705973" velocity="0"/>
-    </joint>
-    <joint type="fixed" name="${prefix}joint_piston">
-      <origin xyz="0.475 0 0" rpy="0 0 0"/>
-      <axis xyz="1 0 0"/>
-      <parent link="${prefix}link_cylinder"/>
-      <child link="${prefix}link_piston"/>
-      <limit effort="0" lower="0" upper="0.6" velocity="0"/>
-    </joint>-->
-    <!-- end of joint list -->
     <!-- ROS base_link to ABB World Coordinates transform -->
     <link name="${prefix}base" />
