Commit message: Collision somewhat working

File: wire_cutting/urdf/irb6400r_macro_parallel.xacro (robot description, xacro)
@@ -109,4 +109,10 @@
     <link name="${prefix}tool0"/>
     <link name="${prefix}carbon_hotwire" >
+      <collision>
+        <geometry>
+          <convex_mesh filename="package://wire_cutting/meshes/carbon_hotwire.stl" />
+        </geometry>
+        <material name="yellow"/>
+      </collision>
       <visual>
         <geometry>
@@ -114,9 +120,4 @@
         </geometry>>
       </visual>
-      <collision>
-        <geometry>
-          <mesh filename="package://wire_cutting/meshes/carbon_hotwire.stl" />
-        </geometry>
-      </collision>
     </link>
     <joint type="revolute" name="${prefix}joint_1">
