Commit message: Reorganized urdf

File: wire_cutting/urdf/irb6400r_parallel_macro.xacro (robot description, xacro)
@@ -1,5 +1,5 @@
 <?xml version="1.0"?>
 <robot xmlns:xacro="http://ros.org/wiki/xacro">
-  <xacro:macro name="irb6400r" params="prefix">
+  <xacro:macro name="irb6400r_robot" params="prefix">
     <!-- link list -->
     <link name="${prefix}base_link">
@@ -108,5 +108,5 @@
     </link>
     <link name="${prefix}tool0"/>
-    <link name="${prefix}carbon_hotwire" >
+    <!--<link name="${prefix}carbon_hotwire" >
       <collision>
         <geometry>
@@ -120,5 +120,5 @@
         </geometry>>
       </visual>
-    </link>
+    </link>-->
     <joint type="revolute" name="${prefix}joint_1">
       <origin xyz="0 0 0.27" rpy="0 0 0"/>
@@ -177,9 +177,9 @@
       <origin xyz=".037 0 0" rpy="0 1.57079632679 0"/>
     </joint>
-    <joint type="fixed" name="${prefix}tool0-carbon_hotwire">
+    <!--<joint type="fixed" name="${prefix}tool0-carbon_hotwire">
       <parent link="${prefix}tool0"/>
       <child link="${prefix}carbon_hotwire"/>
       <origin xyz="0 0 1.861" rpy="0 0 0"/>
-    </joint>
+    </joint>-->
     <!-- ROS base_link to ABB World Coordinates transform -->
     <link name="${prefix}base" />
