Commit message: Hotwire collision geometry

File: wire_cutting/urdf/carbon_hotwire_macro.xacro (robot description, xacro)
@@ -6,5 +6,5 @@
       <collision>
         <geometry>
-          <convex_mesh filename="package://wire_cutting/meshes/carbon_hotwire.stl" convert="true"/>
+          <convex_mesh filename="package://wire_cutting/meshes/CH_top.stl" convert="true"/>
         </geometry>
         <material name="yellow"/>
@@ -12,5 +12,5 @@
       <visual>
         <geometry>
-          <mesh filename="package://wire_cutting/meshes/carbon_hotwire.stl" />
+          <mesh filename="package://wire_cutting/meshes/CH_top.stl" />
         </geometry>>
       </visual>
@@ -21,4 +21,40 @@
   	<origin xyz="0 0 1.861" rpy="0 0 0"/>
   </joint>
+  <link name="${prefix}CH_left" >
+      <collision>
+        <geometry>
+          <convex_mesh filename="package://wire_cutting/meshes/CH_left.stl" convert="true"/>
+        </geometry>
+        <material name="yellow"/>
+      </collision>
+      <visual>
+        <geometry>
+          <mesh filename="package://wire_cutting/meshes/CH_left.stl" />
+        </geometry>>
+      </visual>
+  </link>
+  <link name="${prefix}CH_right" >
+      <collision>
+        <geometry>
+          <convex_mesh filename="package://wire_cutting/meshes/CH_right.stl" convert="true"/>
+        </geometry>
+        <material name="yellow"/>
+      </collision>
+      <visual>
+        <geometry>
+          <mesh filename="package://wire_cutting/meshes/CH_right.stl" />
+        </geometry>>
+      </visual>
+  </link>
+  <joint type="fixed" name="top-left">
+  	<parent link="carbon_hotwire"/>
+  	<child link="CH_left"/>
+  	<origin xyz="0 0 0" rpy="0 0 0"/>
+  </joint>
+  <joint type="fixed" name="top-right">
+  	<parent link="carbon_hotwire"/>
+  	<child link="CH_right"/>
+  	<origin xyz="0 0 0" rpy="0 0 0"/>
+  </joint>
   </xacro:macro>
 </robot>

File: wire_cutting/urdf/wire_cutting_workcell.xacro (robot description, xacro)
@@ -8,5 +8,5 @@
   	<parent link="tool0"/>
   	<child link="carbon_hotwire_mount"/>
-  	<origin xyz="0 0 0" rpy="0 0 0"/>
+  	<origin xyz="0 0 0" rpy="0 0 3.14"/>
   </joint>
 </robot>
