Commit message: costs added

File: wire_cutting/urdf/irb6400r_macro.xacro (robot description, xacro)
@@ -106,4 +106,16 @@
     </link>
     <link name="${prefix}tool0"/>
+    <link name="${prefix}carbon_hotwire" >
+      <visual>
+        <geometry>
+          <mesh filename="package://wire_cutting/meshes/carbon_hotwire.stl" />
+        </geometry>>
+      </visual>
+      <collision>
+        <geometry>
+          <mesh filename="package://wire_cutting/meshes/carbon_hotwire.stl" />
+        </geometry>
+      </collision>
+    </link>
     <!--Cylinder and piston -->
     <!--link name="${prefix}link_cylinder">
@@ -143,5 +155,5 @@
       <parent link="${prefix}base_link"/>
       <child link="${prefix}link_1"/>
-      <limit effort="0" lower="-2.967" upper="2.967" velocity="1.7453"/>
+      <limit effort="0" lower="-3.14" upper="3.14" velocity="1.57"/>
     </joint>
     <joint type="revolute" name="${prefix}joint_2">
@@ -150,5 +162,5 @@
       <parent link="${prefix}link_1"/>
       <child link="${prefix}link_2"/>
-      <limit effort="0" lower="-1.134" upper="1.4855" velocity="1.5707"/>
+      <limit effort="0" lower="-1.22" upper="1.48" velocity="1.22"/>
     </joint>
     <!-- TODO fix 3rd axis geometry -->
@@ -158,5 +170,5 @@
       <parent link="${prefix}link_2"/>
       <child link="${prefix}link_3"/>
-      <limit effort="0" lower="-3.142" upper="1.222" velocity="1.5707"/>
+      <limit effort="0" lower="-0.489" upper="1.92" velocity="1.22"/>
     </joint>
     <!-- TODO find isue with 4-5 axis joint position -->
@@ -166,12 +178,12 @@
       <parent link="${prefix}link_3"/>
       <child link="${prefix}link_4"/>
-      <limit effort="0" lower="-5.236" upper="5.236" velocity="2.9671"/>
+      <limit effort="0" lower="-5.23" upper="5.23" velocity="1.91"/>
     </joint>
     <joint type="revolute" name="${prefix}joint_5">
-      <origin xyz="1.485 0 0 " rpy="0 0 0"/>
+      <origin xyz="1.725 0 0 " rpy="0 0 0"/>
       <axis xyz="0 1 0"/>
       <parent link="${prefix}link_4"/>
       <child link="${prefix}link_5"/>
-      <limit effort="0" lower="-2.094" upper="2.094" velocity="2.4435"/>
+      <limit effort="0" lower="-2.094" upper="2.094" velocity="1.91"/>
     </joint>
      <!-- TODO verify 0.145! -->
@@ -181,5 +193,5 @@
       <parent link="${prefix}link_5"/>
       <child link="${prefix}link_6"/>
-      <limit effort="0" lower="-6.283" upper="6.283" velocity="3.3161"/>
+      <limit effort="0" lower="-5.23" upper="5.23" velocity="1.91"/>
     </joint>
     <joint type="fixed" name="${prefix}joint_6-tool0">
@@ -187,4 +199,9 @@
       <child link="${prefix}tool0"/>
       <origin xyz=".037 0 0" rpy="0 1.57079632679 0"/>
+    </joint>
+    <joint type="fixed" name="${prefix}tool0-carbon_hotwire">
+      <parent link="${prefix}tool0"/>
+      <child link="${prefix}carbon_hotwire"/>
+      <origin xyz="0 0 1.861" rpy="0 0 0"/>
     </joint>
     <!--<joint type="fixed" name="${prefix}joint_cylinder">

Commit message: Basic example working

File: wire_cutting/urdf/irb6400r_macro.xacro (robot description, xacro)
@@ -164,5 +164,4 @@
       <limit effort="0" lower="-1.22" upper="1.48" velocity="1.22"/>
     </joint>
-    <!-- TODO fix 3rd axis geometry -->
     <joint type="revolute" name="${prefix}joint_3">
       <origin xyz="0 0 1.05" rpy="0 0 0"/>
@@ -172,7 +171,6 @@
       <limit effort="0" lower="-0.489" upper="1.92" velocity="1.22"/>
     </joint>
-    <!-- TODO find isue with 4-5 axis joint position -->
     <joint type="revolute" name="${prefix}joint_4">
-      <origin xyz="0 0 0.225" rpy="0 0 0"/>
+      <origin xyz="0.0 0 0.225" rpy="0 0 0"/>
       <axis xyz="1 0 0"/>
       <parent link="${prefix}link_3"/>

Commit message: Basic flow worked out, needs clean up

File: wire_cutting/urdf/irb6400r_macro.xacro (robot description, xacro)
@@ -1,5 +1,5 @@
 <?xml version="1.0"?>
 <robot xmlns:xacro="http://ros.org/wiki/xacro">
-  <xacro:macro name="irb6400r" params="prefix">
+  <xacro:macro name="irb6400r_robot" params="prefix">
     <!-- link list -->
     <link name="${prefix}base_link">
@@ -106,5 +106,11 @@
     </link>
     <link name="${prefix}tool0"/>
-    <link name="${prefix}carbon_hotwire" >
+    <!--<link name="${prefix}carbon_hotwire" >
+      <collision>
+        <geometry>
+          <convex_mesh filename="package://wire_cutting/meshes/carbon_hotwire.stl" />
+        </geometry>
+        <material name="yellow"/>
+      </collision>
       <visual>
         <geometry>
@@ -112,42 +118,5 @@
         </geometry>>
       </visual>
-      <collision>
-        <geometry>
-          <mesh filename="package://wire_cutting/meshes/carbon_hotwire.stl" />
-        </geometry>
-      </collision>
-    </link>
-    <!--Cylinder and piston -->
-    <!--link name="${prefix}link_cylinder">
-      <collision name="collision">
-        <geometry>
-          <mesh filename="package://wire_cutting/meshes/irb6400r/collision/cylinder.stl"/>
-        </geometry>
-        <material name="yellow"/>
-      </collision>
-      <visual name="visual">
-        <geometry>
-          <mesh filename="package://wire_cutting/meshes/irb6400r/visual/cylinder.stl"/>
-        </geometry>
-        <material name="orange"/>
-      </visual>
-    </link>
-    <link name="${prefix}link_piston">
-      <collision name="collision">
-        <geometry>
-          <mesh filename="package://wire_cutting/meshes/irb6400r/collision/piston.stl"/>
-        </geometry>
-        <material name="yellow"/>
-      </collision>
-      <visual name="visual">
-        <geometry>
-          <mesh filename="package://wire_cutting/meshes/irb6400r/visual/piston.stl"/>
-        </geometry>
-        <material name="orange"/>
-      </visual>
-    </link> -->
-    <!-- end of link list -->
-    <!-- joint list -->
-    <!-- TODO update limits and velocities (bar linkage between axis 2 and 3!)-->
+    </link>-->
     <joint type="revolute" name="${prefix}joint_1">
       <origin xyz="0 0 0.27" rpy="0 0 0"/>
@@ -169,5 +138,5 @@
       <parent link="${prefix}link_2"/>
       <child link="${prefix}link_3"/>
-      <limit effort="0" lower="-0.489" upper="1.92" velocity="1.22"/>
+      <limit effort="0" lower="-3.14" upper="3.14" velocity="1.22"/> <!-- Limits defined by constraints due to parallel link-->
     </joint>
     <joint type="revolute" name="${prefix}joint_4">
@@ -198,24 +167,9 @@
       <origin xyz=".037 0 0" rpy="0 1.57079632679 0"/>
     </joint>
-    <joint type="fixed" name="${prefix}tool0-carbon_hotwire">
+    <!--<joint type="fixed" name="${prefix}tool0-carbon_hotwire">
       <parent link="${prefix}tool0"/>
       <child link="${prefix}carbon_hotwire"/>
       <origin xyz="0 0 1.861" rpy="0 0 0"/>
-    </joint>
-    <!--<joint type="fixed" name="${prefix}joint_cylinder">
-      <origin xyz="-0.365 -0.1895 0.405" rpy="0 -0.170 0"/>
-      <axis xyz="0 1 0"/>
-      <parent link="${prefix}link_1"/>
-      <child link="${prefix}link_cylinder"/>
-      <limit effort="0" lower="-2.96705973" upper="2.96705973" velocity="0"/>
-    </joint>
-    <joint type="fixed" name="${prefix}joint_piston">
-      <origin xyz="0.475 0 0" rpy="0 0 0"/>
-      <axis xyz="1 0 0"/>
-      <parent link="${prefix}link_cylinder"/>
-      <child link="${prefix}link_piston"/>
-      <limit effort="0" lower="0" upper="0.6" velocity="0"/>
     </joint>-->
-    <!-- end of joint list -->
     <!-- ROS base_link to ABB World Coordinates transform -->
     <link name="${prefix}base" />

File: wire_cutting/urdf/wire_cutting_workcell.xacro (robot description, xacro)
@@ -1,5 +1,5 @@
 <?xml version="1.0" ?>
 <robot name="irb6400r" xmlns:xacro="http://wiki.ros.org/xacro">
-  <xacro:include filename="$(find wire_cutting)/urdf/irb6400r_parallel_macro.xacro" />
+  <xacro:include filename="$(find wire_cutting)/urdf/irb6400r_macro.xacro" />
   <xacro:include filename="$(find wire_cutting)/urdf/carbon_hotwire_macro.xacro" />
   <xacro:irb6400r_robot prefix=""/>

Commit message: Test cases

File: wire_cutting/urdf/irb6400r_macro.xacro (robot description, xacro)
@@ -3,4 +3,30 @@
   <xacro:macro name="irb6400r_robot" params="prefix">
     <!-- link list -->
+   <link name="${prefix}floor" >
+      <collision>
+        <geometry>
+          <convex_mesh filename="package://wire_cutting/meshes/Floor.stl" convert="true"/>
+        </geometry>
+        <material name="yellow"/>
+      </collision>
+      <visual>
+        <geometry>
+          <mesh filename="package://wire_cutting/meshes/Floor.stl" />
+        </geometry>>
+      </visual>
+   </link>
+    <link name="${prefix}pedestal" >
+      <collision>
+        <geometry>
+          <convex_mesh filename="package://wire_cutting/meshes/Pedestal.stl" convert="true"/>
+        </geometry>
+        <material name="yellow"/>
+      </collision>
+      <visual>
+        <geometry>
+          <mesh filename="package://wire_cutting/meshes/Pedestal.stl" />
+        </geometry>>
+      </visual>
+   </link>
     <link name="${prefix}base_link">
       <collision name="collision">
@@ -179,4 +205,14 @@
       <child link="${prefix}base"/>
     </joint>
+    <joint name="${prefix}base_pedestal" type="fixed">
+      <origin xyz="0 0 0" rpy="0 0 0"/>
+      <parent link="${prefix}base"/>
+      <child link="${prefix}pedestal"/>
+    </joint>
+    <joint name="${prefix}base_fllor" type="fixed">
+      <origin xyz="0 0 0" rpy="0 0 0"/>
+      <parent link="${prefix}base"/>
+      <child link="${prefix}floor"/>
+    </joint>
   </xacro:macro>
 </robot>

Commit message: new

File: wire_cutting/urdf/irb6400r_macro.xacro (robot description, xacro)
@@ -210,5 +210,5 @@
       <child link="${prefix}pedestal"/>
     </joint>
-    <joint name="${prefix}base_fllor" type="fixed">
+    <joint name="${prefix}base_floor" type="fixed">
       <origin xyz="0 0 0" rpy="0 0 0"/>
       <parent link="${prefix}base"/>

Commit message: small changes

File: wire_cutting/urdf/irb6400r_macro.xacro (robot description, xacro)
@@ -164,5 +164,5 @@
       <parent link="${prefix}link_2"/>
       <child link="${prefix}link_3"/>
-      <limit effort="0" lower="-3.14" upper="3.14" velocity="1.22"/> <!-- Limits defined by constraints due to parallel link-->
+      <limit effort="0" lower="-1.57" upper="1.57" velocity="1.22"/> <!-- Limits defined by constraints due to parallel link-->
     </joint>
     <joint type="revolute" name="${prefix}joint_4">
